File: sensorShield/sensorShield.sch (KiCad schematic (older format))
At the start: 18 parts, among them P1 Power, P2 Analog, P3 Digital, P4 Digital, P5 CONN_01X01, P6 CONN_01X01, P7 CONN_01X01, P8 CONN_01X01

Commit message: sensor schematized
Parts:
- added U2: GrooveConnector, Connector_PinSocket_2.00mm:PinSocket_1x04_P2.00mm_Vertical, symbol Sensor_Gas:GrooveConnector
- added U3: RN2483, symbol RN2483:RN2483_Breakout
- gave numbers to parts that had none: 1
Connections:
- net labels added: Rx, Tx
- wire segments 73 -> 80
- no-connect marks 5 -> 14
Other:
- moved on the sheet: C1, C2, C3, C4, R3, R4, R5, R6, R7
