File: sensorShield/sensorShield.sch (KiCad schematic (older format))
At the start: 20 parts, among them P1 Power, P2 Analog, P3 Digital, P4 Digital, P5 CONN_01X01, P6 CONN_01X01, P7 CONN_01X01, P8 CONN_01X01, U1 AOPSENSOR, U2 GrooveConnector, U3 RN2483

Commit message: KiCad push
Parts:
- removed P1: Power, Socket_Arduino_Uno:Socket_Strip_Arduino_1x08, symbol Connector_Generic:Conn_01x08
- removed P2: Analog, Socket_Arduino_Uno:Socket_Strip_Arduino_1x06, symbol Connector_Generic:Conn_01x06
- removed P3: Digital, Socket_Arduino_Uno:Socket_Strip_Arduino_1x10, symbol Connector_Generic:Conn_01x10
- removed P4: Digital, Socket_Arduino_Uno:Socket_Strip_Arduino_1x08, symbol Connector_Generic:Conn_01x08
- removed P5, P6, P7, P8: CONN_01X01, Socket_Arduino_Uno:Arduino_1pin, symbol Connector_Generic:Conn_01x01
- removed U1: AOPSENSOR, symbol aopsensor:AOPSENSOR
- removed U2: GrooveConnector, Connector_PinSocket_2.00mm:PinSocket_1x04_P2.00mm_Vertical, symbol Sensor_Gas:GrooveConnector
- removed U3: RN2483, symbol RN2483:RN2483_Breakout
- added A?: Arduino_UNO_R3, Module:Arduino_UNO_R3, symbol MCU_Module:Arduino_UNO_R3
- added D1: LED, LED_THT:LED_D3.0mm, symbol Device:LED
- added J2: GrooveGasSensor, Connector_PinHeader_2.00mm:PinHeader_1x04_P2.00mm_Vertical, symbol Connector_Generic:Conn_01x04
- added R1: 10k, Resistor_THT:R_Axial_DIN0204_L3.6mm_D1.6mm_P7.62mm_Horizontal, symbol Device:R
- added R2: 330, Resistor_THT:R_Axial_DIN0204_L3.6mm_D1.6mm_P7.62mm_Horizontal, symbol Device:R
- added SW1: SW_Push, Button_Switch_THT:SW_PUSH_6mm, symbol Switch:SW_Push
- added U1: RN2483, RF_Module:RN42N, symbol RF_Lora:RN2483
- added U2: LTC1050, symbol Amplifier_Operational:LTC1050
- added U3: GazSensor, Package_TO_SOT_THT:TO-5-8, symbol gasSensor:GazSensor-SensorGaz
- C1: value C -> 100n; footprint (none) -> Capacitor_THT:C_Axial_L3.8mm_D2.6mm_P7.50mm_Horizontal
- C2: footprint (none) -> Capacitor_THT:C_Rect_L7.0mm_W4.5mm_P5.00mm
- C3, C4: footprint (none) -> Capacitor_THT:C_Axial_L3.8mm_D2.6mm_P7.50mm_Horizontal
- R3, R4, R5, R6, R7: footprint (none) -> Resistor_THT:R_Axial_DIN0204_L3.6mm_D1.6mm_P7.62mm_Horizontal
Connections:
- net labels added: +3V3, CapTemp, D2, D3, RChauff, RST
- net labels removed: 0(Rx), 1(Tx), 10(**/SS), 11(**/MOSI), 12(MISO), 13(SCK), 2, 3(**), 4, 5(**), 6(**), 7, 8, 9(**), A2, A3, A4(SDA), A5(SCL), AREF, IOREF, Reset, Vin
- no-connect marks 23 -> 24
Other:
- note removed: "1"
- note removed: "Holes"
- note removed: "Shield for Arduino that uses\nthe same pin disposition\nlike "Uno" board Rev 3."
